Commit message: Added trashcan and robot listens to change state
Listens to real microphone using vosk because Gazebo doesn't support sounds as I need them to be represented

File: src/smartbin_robot/urdf/base_link.urdf.xacro (robot description, xacro)
@@ -28,8 +28,34 @@
       <origin xyz="${xyz}" rpy="${rpy}" />
     </joint>
+    <!-- Trash Can Link -->
+    <link name="trashcan_link">
+      <visual>
+        <geometry>
+          <cylinder radius="0.09" length="0.3"/>
+        </geometry>
+        <material name="grey">
+          <color rgba="0.5 0.5 0.5 1.0"/>
+        </material>
+      </visual>
+      <collision>
+        <geometry>
+          <cylinder radius="0.09" length="0.3"/>
+        </geometry>
+      </collision>
+      <inertial>
+        <mass value="1.0" />
+        <inertia ixx="0.02" ixy="0.0" ixz="0.0" iyy="0.02" iyz="0.0" izz="0.01"/>
+      </inertial>
+    </link>
+    <joint name="trashcan_joint" type="fixed">
+      <parent link="base_link"/>
+      <child link="trashcan_link"/>
+      <origin xyz="-0.025 0 0.24" rpy="0 0 0"/>
+    </joint>
+    <!-- Omni Wheels -->
     <xacro:omni_wheel parent="base_link" suffix="1" xyz="0.0927 0.0000 0.0145" rpy="-0.8040 1.5708 -0.8040"/>
     <xacro:omni_wheel parent="base_link" suffix="2" xyz="-0.0464 0.0803 0.0145" rpy="-0.8040 1.5708 1.290"/>
     <xacro:omni_wheel parent="base_link" suffix="3" xyz="-0.0464 -0.0803 0.0145" rpy="-0.8040 1.5708 -2.8984"/>
-    <!-- Sensors: Calls to the macros defined in main.urdf.xacro -->
+    <!-- Sensors -->
     <xacro:camera parent="base_link" suffix="1" xyz="0.1035 -0.0000 0.0630" rpy="0 0 0"/>
     <xacro:lidar parent="base_link" suffix="1" xyz="0.1000 0.0000 0.1000" rpy="0 0 0"/>

Commit message: Much better pathing

File: src/smartbin_robot/urdf/base_link.urdf.xacro (robot description, xacro)
@@ -18,7 +18,7 @@
         <mass value="3.0" />
         <inertia
-          ixx="0.9" ixy="0.0" ixz="0.0"
-          iyy="0.9" iyz="0.0"
-          izz="0.01"/>
+          ixx="0.02" ixy="0.0" ixz="0.0"
+          iyy="0.02" iyz="0.0"
+          izz="0.04"/>
       </inertial>
     </link>

File: src/smartbin_robot/urdf/omni_wheel.urdf.xacro (robot description, xacro)
@@ -13,6 +13,7 @@
       </visual>
       <collision>
+        <origin xyz="0 0 0" rpy="0 0 0"/>
         <geometry>
-          <mesh filename="package://smartbin_robot/meshes/omni_frame.stl" />
+          <cylinder radius="0.03" length="0.015"/>
         </geometry>
       </collision>

Commit message: Visual update, map update, cleaning comments

File: src/smartbin_robot/urdf/base_link.urdf.xacro (robot description, xacro)
@@ -31,16 +31,9 @@
     <link name="trashcan_link">
       <visual>
+      <origin xyz="0 0 -0.15" rpy="1.5708 0 1.5708" />
         <geometry>
-          <cylinder radius="0.09" length="0.3"/>
+          <mesh filename="package://smartbin_robot/meshes/Rubbish_Bin_By_Berken.dae" scale="0.13 0.13 0.13"/>
         </geometry>
-        <material name="grey">
-          <color rgba="0.5 0.5 0.5 1.0"/>
-        </material>
       </visual>
-      <collision>
-        <geometry>
-          <cylinder radius="0.09" length="0.3"/>
-        </geometry>
-      </collision>
       <inertial>
         <mass value="1.0" />

File: src/smartbin_robot/urdf/lidar.urdf.xacro (robot description, xacro)
@@ -7,6 +7,6 @@
           <cylinder radius="0.02" length="0.02" />
         </geometry>
-        <material name="red">
-          <color rgba="0.4 0 0.1 1" />
+        <material name="blue">
+          <color rgba="0.03 0.075 0.3 1" />
         </material>
       </visual>
